File: pcb/MI0283QT_v20.brd (EAGLE design)
At the start: 52 x 85 mm, 52 parts, among them Q1 16MHz, T1 N-CHN, U1 TS5204, X1 PASSER, X2 PASSER, X3 PASSER, X4 PASSER

Commit message: updated schematic and layout files
Parts:
- U1: value TS5204 -> TS5204-3V3
Changed lines of the file:
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@@
 <?xml version="1.0" encoding="utf-8"?>
 <!DOCTYPE eagle SYSTEM "eagle.dtd">
-<eagle version="6.5.0">
+<eagle version="6.6.0">
 <drawing>
 <settings>
@@
 <attribute name="NAME" x="7.4613" y="30.7975" size="0.8128" layer="26" font="vector" ratio="10" rot="MR180"/>
 </element>
-<element name="U1" library="Voltage-Reg" package="SOT23" value="TS5204" x="15.875" y="8.255" smashed="yes" rot="MR0">
+<element name="U1" library="Voltage-Reg" package="SOT23" value="TS5204-3V3" x="15.875" y="8.255" smashed="yes" rot="MR0">
 <attribute name="NAME" x="16.51" y="10.3188" size="0.8128" layer="26" font="vector" ratio="10" rot="MR0"/>
 <attribute name="VALUE" x="18.0975" y="11.6841" size="0.8128" layer="28" font="vector" ratio="10" rot="MR0"/>
