File: pcb/MI0283QT_v14.brd (EAGLE design)
At the start: 52 x 85 mm, 52 parts, among them Q1 16MHz, T1 N-CHN, U1 TS5204-3V3, X1 PASSER, X2 PASSER, X3 PASSER, X4 PASSER

Commit message: updated layout and schematics
Parts:
- removed 1-GND, 2-CTS, 3-VCC, 4-TXO, 5-RXI, 6-DTR: WIREPADSMD1,27-254, wirepad:SMD1,27-2,54
- removed ARM: LPC1114FBD48, ARM:LQFP48
- removed ISP, RST, RXD, TXD, VCC: (no value), jumper:SJ
- removed LDR+, LDR-, LED+, LED-: WIREPAD2,15/1,0, wirepad:2,15/1,0
- removed Q1: 16MHz, Crystal:SMD_OSC_35X15
- removed R10, R7, R8, R9: 22, rcl:R0603
- removed SW_ISP: SW_SMDS, Switch-SMD:SW_SMD4@1
- added BUSY-RS, IM0, IM1: (no value), jumper:SJ_2
- added C9: 100nF, rcl:C0603
- added IC1: ADS7846, Display:SSOP16
- added IC2: 74LVC244, 74xx-eu:SO20W
- added R16: 100k, rcl:R0603
- added VREF-3V3: (no value), jumper:SJ
- CON1: device con-lstb:MA10-2 -> con-lsta:FE08-2
- R1, R2, R3, R4, R5: value 22 -> 47
- R12, R13, R14: value 10k -> 100k
- R15: value 1k -> 100k
- moved R13 50.1 mm to (13.6, 47.0), turned to 180 degrees
- moved R12 33.3 mm to (-3.81, 39.4), turned to 0 degrees
- moved R14 21.5 mm to (-17.9, 35.1)
- moved R15 16.2 mm to (-14.6, 43.2), turned to 0 degrees
- moved C5 16.2 mm to (-17.9, 38.0)
- moved C6 8.91 mm to (20.0, 36.7)
- moved R11 4.33 mm to (-3.81, 47.0), turned to 0 degrees
- moved C7 4.10 mm to (-3.81, 50.5)
- moved C4 3.17 mm to (5.08, 36.2), turned to 0 degrees
- moved CON1 2.54 mm to (0.00, 4.45), flipped to the bottom, turned to 0 degrees
- turned CON2 to 0 degrees
Connections:
- removed net AD4: ARM.39, CON1.15, LDR+.1
- removed net AD5: ARM.40, C7.1, LDR-.1, R14.2
- removed net AD7: ARM.42, CON1.16
- removed net CS: ARM.10, CON1.7
- removed net C_ISP: CON2.1, ISP.1
- removed net C_RST: CON2.8, RST.1
- removed net C_RXD: CON2.6, RXD.1
- removed net C_TXD: CON2.7, TXD.1
- removed net C_VCC: CON2.5, VCC.1
- removed net GPIO: ARM.14, CON1.5
- removed net ISP: ARM.4, ISP.2, SW_ISP.1, SW_ISP.4
- removed net LCD_D0: ARM.2, LCD.32
- removed net LCD_D1: ARM.13, LCD.31
- removed net LCD_D2: ARM.26, LCD.30
- removed net LCD_D3: ARM.38, LCD.29
- removed net LCD_D4: ARM.19, LCD.28
- removed net LCD_D5: ARM.20, LCD.27
- removed net LCD_D6: ARM.1, LCD.26
- removed net LCD_D7: ARM.11, LCD.25
- removed net LCD_RD: ARM.21, LCD.35
- removed net LCD_WR: ARM.24, LCD.36
- removed net LED: ARM.36, R15.1
- removed net MISO: ARM.27, CON1.9
- removed net MOSI: ARM.28, CON1.8
- removed net N$8: LED+.1, R15.2
- removed net RST: 6-DTR.1, ARM.3, CON1.6, R11.1, RST.2
- removed net RXD: 4-TXO.1, ARM.46, CON1.12, RXD.2
- removed net SCK: ARM.29, CON1.10
- removed net SDA: ARM.16, CON1.14, R13.1
- removed net TXD: 5-RXI.1, ARM.47, CON1.11, TXD.2
- removed net X+: ARM.32, R7.2
- removed net X-: ARM.34, R8.2
- removed net XM: LCD.46, R8.1
- removed net XP: LCD.44, R7.1
- removed net Y+: ARM.33, R9.2
- removed net Y-: ARM.35, R10.2
- removed net YM: LCD.47, R10.1
- removed net YP: LCD.45, R9.1
- new net A-ADS_BUSY: IC1.13, IC2.15, R14.1
- new net A-ADS_CS: CON1.11, IC2.13, R13.1
- new net A-ADS_IRQ: IC1.11, IC2.17, R15.1
- new net A-LCD_CS: CON1.7, IC2.2, R12.1
- new net A-LCD_RS: BUSY-RS.3, IC2.6
- new net A-LCD_RST: CON1.6, IC2.8, R11.1
- new net A-SCL: CON1.10, IC2.11
- new net A-SDI: CON1.8, IC2.4
- new net ADS_AUX: CON1.14, IC1.8
- new net ADS_BUSY: BUSY-RS.1, IC2.5
- new net ADS_CS: IC1.15, IC2.7
- new net ADS_IRQ: CON1.13, IC2.3
- new net ADS_VBAT: CON1.15, IC1.7
- new net ADS_VREF: C9.1, CON1.16, IC1.9, VREF-3V3.2
- new net IM0: IM0.2, LCD.6
- new net N$3: IC1.4, LCD.46
- new net N$4: IC1.2, LCD.44
- new net N$5: IM1.2, LCD.7
- new net N$6: BUSY-RS.2, CON1.12
- new net SDI: IC1.14, IC2.16, LCD.34
- new net SDO: CON1.9, IC1.12, LCD.33
- net +3V3: now also C7.1, IC1.1, IC1.10, IC2.20, IM0.3, IM1.3, LCD.8, LCD.9, R15.2, VREF-3V3.1; no longer ARM.44, ARM.8
- net GND: now also C9.2, CON2.1, CON2.5, CON2.6, CON2.7, CON2.8, IC1.6, IC2.1, IC2.10, IC2.19, IM0.1, IM1.1, LCD.25, LCD.26, LCD.27, LCD.28, LCD.29, LCD.30, LCD.31, LCD.32, LCD.35, LCD.39, R14.2, R16.2; no longer 1-GND.1, 2-CTS.1, ARM.41, ARM.5, CON1.19, CON1.20, LCD.34, LCD.6, LCD.7, LCD.8, LCD.9, LED-.1, Q1.GND, R14.1, SW_ISP.2, SW_ISP.3
- net LCD_CS: now also IC2.18; no longer ARM.31
- net LCD_LED: now also CON1.5; no longer ARM.17
- net LCD_RS: now also IC2.14, LCD.36; no longer ARM.25, LCD.37
- net LCD_RST: now also IC2.12; no longer ARM.12
- net N$1: now also IC1.5, LCD.47; no longer ARM.6, Q1.2
- net N$2: now also IC1.3, LCD.45; no longer ARM.7, Q1.1
- net SCL: now also IC1.16, IC2.9, LCD.37; no longer ARM.15, CON1.13, R12.1
- net VCC: no longer 3-VCC.1, CON1.17, CON1.18, VCC.2
Routing:
- net RXD: track 124.6 -> 0.00 mm, vias 2 -> 0
- net RST: track 120.2 -> 0.00 mm
- net TXD: track 118.1 -> 0.00 mm, vias 2 -> 0
- net A-LCD_RS: track 0.00 -> 109.7 mm
- net AD4: track 101.7 -> 0.00 mm, vias 3 -> 0
- net A-LCD_RST: track 0.00 -> 88.8 mm, vias 0 -> 1
- net A-SDI: track 0.00 -> 88.0 mm, vias 0 -> 3
- net VCC: track 153.3 -> 69.0 mm, vias 4 -> 0
- net A-ADS_CS: track 0.00 -> 77.8 mm, vias 0 -> 2
- net A-SCL: track 0.00 -> 76.1 mm, vias 0 -> 1
- net SDO: track 0.00 -> 75.8 mm, vias 0 -> 2
- net GPIO: track 74.2 -> 0.00 mm, vias 2 -> 0
- net SDA: track 73.6 -> 0.00 mm, vias 2 -> 0
- net SCL: track 105.2 -> 33.3 mm, vias 3 -> 2
- net CS: track 71.9 -> 0.00 mm, vias 2 -> 0
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Other:
- board text added: "Aux"
- board text added: "Busy"
- board text added: "Display"
- board text added: "IRQ"
- board text added: "LED"
- board text added: "Rev 1.4"
- board text added: "SDI"
- board text added: "SDO"
- board text added: "Touch"
- board text added: "VBat"
- board text added: "VRef"
- board text removed: "AD4"
- board text removed: "AD7"
- board text removed: "DTR"
- board text removed: "FTDI-Connector"
- board text removed: "IO"
- board text removed: "MISO"
- board text removed: "MOSI"
- board text removed: "Rev 2.0"
- board text removed: "Rx"
- board text removed: "SCK"
- board text removed: "SDA"
- board text removed: "Tx"
- board text removed: "blk"
- board text removed: "grn"
- board text removed: "o"
