File: pcb/MI0283QT_v10.brd (EAGLE design)
At the start: 52 x 85 mm, 35 parts, among them IC1 ADS7846, IC2 74LVC244, Q1 N-CHN, U1 TS5204, X1 PASSER, X2 PASSER, X3 PASSER, X4 PASSER

Commit message: updated license infos
Parts:
- R1, R2, R3, R4, R5: value 22 -> 47
Changed lines of the file:
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@@
 <elements>
 <element name="LCD" library="Display" package="MI0283QT" value="MI0283QT" x="-25.0825" y="8.89" smashed="yes"/>
-<element name="R1" library="rcl" package="R0603" value="22" x="19.685" y="29.845" smashed="yes" rot="MR90">
+<element name="R1" library="rcl" package="R0603" value="47" x="19.685" y="29.845" smashed="yes" rot="MR90">
 <attribute name="NAME" x="18.7923" y="27.5272" size="0.8128" layer="26" font="vector" rot="MR180"/>
 </element>
-<element name="R2" library="rcl" package="R0603" value="22" x="17.4625" y="29.845" smashed="yes" rot="MR90">
+<element name="R2" library="rcl" package="R0603" value="47" x="17.4625" y="29.845" smashed="yes" rot="MR90">
 <attribute name="NAME" x="16.7285" y="27.5272" size="0.8128" layer="26" font="vector" rot="MR180"/>
 </element>
-<element name="R3" library="rcl" package="R0603" value="22" x="15.24" y="29.845" smashed="yes" rot="MR90">
+<element name="R3" library="rcl" package="R0603" value="47" x="15.24" y="29.845" smashed="yes" rot="MR90">
 <attribute name="NAME" x="14.506" y="27.5272" size="0.8128" layer="26" font="vector" rot="MR180"/>
 </element>
-<element name="R4" library="rcl" package="R0603" value="22" x="13.0175" y="29.845" smashed="yes" rot="MR90">
+<element name="R4" library="rcl" package="R0603" value="47" x="13.0175" y="29.845" smashed="yes" rot="MR90">
 <attribute name="NAME" x="12.1247" y="27.5272" size="0.8128" layer="26" font="vector" rot="MR180"/>
 </element>
@@
 <attribute name="VALUE" x="-16.764" y="9.017" size="0.8128" layer="28" font="vector" rot="MR180"/>
 </element>
-<element name="R5" library="rcl" package="R0603" value="22" x="21.9075" y="29.845" smashed="yes" rot="MR90">
+<element name="R5" library="rcl" package="R0603" value="47" x="21.9075" y="29.845" smashed="yes" rot="MR90">
 <attribute name="NAME" x="21.1773" y="27.5273" size="0.8128" layer="26" font="vector" rot="MR180"/>
 <attribute name="VALUE" x="23.0505" y="29.2735" size="0.8128" layer="28" font="vector" rot="MR90"/>

Commit message: updated schematic and layout files
Parts:
- U1: value TS5204 -> TS5204-3V3
Changed lines of the file:
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@@
 <?xml version="1.0" encoding="utf-8"?>
 <!DOCTYPE eagle SYSTEM "eagle.dtd">
-<eagle version="6.5.0">
+<eagle version="6.6.0">
 <drawing>
 <settings>
@@
 <attribute name="NAME" x="12.1247" y="27.5272" size="0.8128" layer="26" font="vector" rot="MR180"/>
 </element>
-<element name="U1" library="Voltage-Reg" package="SOT23" value="TS5204" x="0" y="31.115" smashed="yes" rot="MR180">
+<element name="U1" library="Voltage-Reg" package="SOT23" value="TS5204-3V3" x="0" y="31.115" smashed="yes" rot="MR180">
 <attribute name="NAME" x="-0.635" y="28.8291" size="0.8128" layer="26" font="vector" rot="MR180"/>
 <attribute name="VALUE" x="-2.2225" y="27.6859" size="0.8128" layer="28" font="vector" rot="MR180"/>
