File: pcb/MI0283QT_v10.sch (EAGLE design)
At the start: 35 parts, among them IC1 ADS7846, IC2 74LVC244, Q1 N-CHN, U1 TS5204, X1 PASSER, X2 PASSER, X3 PASSER, X4 PASSER

Commit message: updated license infos
Parts:
- R1, R2, R3, R4, R5: value 22 -> 47
Other:
- note added: "Released under the Creative Commons Attribution Share-Alike License"
- note added: "http://creativecommons.org/licenses/by-sa/4.0/"
- note removed: "Released under the Creative Commons Attribution Share-Alike 3.0 License"
- note removed: "http://creativecommons.org/licenses/by-sa/3.0/"
Changed lines of the file:
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@@
 <part name="LCD" library="Display" deviceset="MI0283QT" device=""/>
 <part name="GND3" library="supply1" deviceset="GND" device=""/>
-<part name="R1" library="rcl" deviceset="R-EU_" device="R0603" value="22"/>
-<part name="R2" library="rcl" deviceset="R-EU_" device="R0603" value="22"/>
-<part name="R3" library="rcl" deviceset="R-EU_" device="R0603" value="22"/>
-<part name="R4" library="rcl" deviceset="R-EU_" device="R0603" value="22"/>
+<part name="R1" library="rcl" deviceset="R-EU_" device="R0603" value="47"/>
+<part name="R2" library="rcl" deviceset="R-EU_" device="R0603" value="47"/>
+<part name="R3" library="rcl" deviceset="R-EU_" device="R0603" value="47"/>
+<part name="R4" library="rcl" deviceset="R-EU_" device="R0603" value="47"/>
 <part name="U1" library="Voltage-Reg" deviceset="TS5204" device=""/>
 <part name="+3V6" library="supply1" deviceset="+3V3" device=""/>
@@
 <part name="C5" library="rcl" deviceset="C-EU" device="C0603" value="100nF"/>
 <part name="C6" library="rcl" deviceset="C-EU" device="C0603" value="100nF"/>
-<part name="R5" library="rcl" deviceset="R-EU_" device="R0603" value="22"/>
+<part name="R5" library="rcl" deviceset="R-EU_" device="R0603" value="47"/>
 <part name="IC1" library="Display" deviceset="ADS7846" device=""/>
 <part name="+3V1" library="supply1" deviceset="+3V3" device=""/>
@@
 <text x="45.085" y="149.225" size="1.778" layer="95">0</text>
 <text x="45.085" y="141.605" size="1.778" layer="95">0</text>
-<text x="161.29" y="31.75" size="1.27" layer="95">Released under the Creative Commons Attribution Share-Alike 3.0 License</text>
-<text x="161.29" y="29.21" size="1.27" layer="95">http://creativecommons.org/licenses/by-sa/3.0/</text>
+<text x="161.29" y="31.75" size="1.27" layer="95">Released under the Creative Commons Attribution Share-Alike License</text>
+<text x="161.29" y="29.21" size="1.27" layer="95">http://creativecommons.org/licenses/by-sa/4.0/</text>
 <text x="161.29" y="25.4" size="1.27" layer="95">Designed by Andreas Watterott (Watterott electronic)</text>
 <text x="44.45" y="166.37" size="3.81" layer="250">Display</text>

Commit message: updated schematic and layout files
Parts:
- U1: value TS5204 -> TS5204-3V3
Changed lines of the file:
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@@
 <?xml version="1.0" encoding="utf-8"?>
 <!DOCTYPE eagle SYSTEM "eagle.dtd">
-<eagle version="6.5.0">
+<eagle version="6.6.0">
 <drawing>
 <settings>
@@
 <part name="R3" library="rcl" deviceset="R-EU_" device="R0603" value="47"/>
 <part name="R4" library="rcl" deviceset="R-EU_" device="R0603" value="47"/>
-<part name="U1" library="Voltage-Reg" deviceset="TS5204" device=""/>
+<part name="U1" library="Voltage-Reg" deviceset="TS5204" device="" value="TS5204-3V3"/>
 <part name="+3V6" library="supply1" deviceset="+3V3" device=""/>
 <part name="GND9" library="supply1" deviceset="GND" device=""/>
