File: pcb/MI0283QT_v11.brd (EAGLE design)
At the start: 52 x 85 mm, 36 parts, among them IC1 ADS7846, IC2 74LVC244, Q1 N-CHN, U1 TS5204, X1 PASSER, X2 PASSER, X3 PASSER, X4 PASSER

Commit message: updated schematic and layout files
Parts:
- U1: value TS5204 -> TS5204-3V3
Changed lines of the file:
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@@
 <?xml version="1.0" encoding="utf-8"?>
 <!DOCTYPE eagle SYSTEM "eagle.dtd">
-<eagle version="6.5.0">
+<eagle version="6.6.0">
 <drawing>
 <settings>
@@
 <attribute name="NAME" x="12.1247" y="27.5272" size="0.8128" layer="26" font="vector" rot="MR180"/>
 </element>
-<element name="U1" library="Voltage-Reg" package="SOT23" value="TS5204" x="0" y="31.115" smashed="yes" rot="MR180">
+<element name="U1" library="Voltage-Reg" package="SOT23" value="TS5204-3V3" x="0" y="31.115" smashed="yes" rot="MR180">
 <attribute name="NAME" x="-0.635" y="28.8291" size="0.8128" layer="26" font="vector" rot="MR180"/>
 <attribute name="VALUE" x="-2.2225" y="27.6859" size="0.8128" layer="28" font="vector" rot="MR180"/>
