File: pcb/MI0283QT_v12b.brd (EAGLE design)
At the start: 52 x 85 mm, 36 parts, among them IC1 ADS7846, IC2 74LVC244, Q1 N-CHN, U1 TS5204, X1 PASSER, X2 PASSER, X3 PASSER, X4 PASSER

Commit message: updated cad files to Eagle xml format
Parts:
- removed ID(0): (no value), jumper:SJ_2
- added BUSY-RS, IM0, IM1: (no value), jumper:SJ_2
- CON2: device con-lsta:FE08 -> con-lstb:MA08-1
- moved R8 19.2 mm to (21.4, 33.8), turned to 90 degrees
- moved R5 0.48 mm to (21.4, 29.8)
- moved C8 0.35 mm to (16.2, 33.8), turned to 90 degrees
- moved Q1 0.32 mm to (20.3, 24.8)
- moved R1 0.32 mm to (19.4, 29.8)
- moved R2 0.16 mm to (17.3, 29.8)
- moved R4 0.16 mm to (13.2, 29.8)
- turned CON2 to 180 degrees
Connections:
- removed net A-LCD_LED: CON1.5, IC2.6, R8.1
- new net A-LCD_RS: BUSY-RS.3, IC2.6
- new net LCD_RS: IC2.14, LCD.36
- new net N$2: BUSY-RS.2, CON1.12
- new net N$4: IM1.2, LCD.9
- net +3V3: now also IM0.3, IM1.3; no longer ID(0).3
- net ADS_BUSY: now also BUSY-RS.1; no longer CON1.12
- net GND: now also IM0.1, IM1.1; no longer CON2.1, CON2.2, CON2.3, CON2.4, CON2.8, ID(0).1, LCD.37, LCD.9
- net IM0: now also IM0.2; no longer ID(0).2
- net LCD_LED: now also CON1.5, R8.1; no longer IC2.14
- net SCL: now also LCD.37; no longer LCD.36
Routing:
- net LCD_RS: track 0.00 -> 22.2 mm, vias 0 -> 1
- net N$2: track 0.00 -> 21.6 mm, vias 0 -> 1
- net A-LCD_RS: track 0.00 -> 18.3 mm, vias 0 -> 2
- net A-LCD_LED: track 16.9 -> 0.00 mm
- net ADS_BUSY: track 30.2 -> 13.6 mm, vias 1 -> 2
- net LCD_LED: track 35.3 -> 50.0 mm, vias 2 -> 1
- net N$4: track 0.00 -> 11.0 mm, vias 0 -> 1
- net VCC: track 81.0 -> 76.7 mm
- net IM0: track 12.0 -> 10.4 mm
- net N$1: track 0.00 -> 1.43 mm
- net N$3: track 0.00 -> 1.43 mm
- net LCD_CS: track 15.0 -> 15.8 mm
Other:
- board text added: "MI0283QT-9A Adapter Rev 1.2b"
- board text removed: "MI0283QT-2 Adapter Rev 1.1"

Commit message: updated schematic and layout files
Parts:
- U1: value TS5204 -> TS5204-3V3
Changed lines of the file:
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@@
 <?xml version="1.0" encoding="utf-8"?>
 <!DOCTYPE eagle SYSTEM "eagle.dtd">
-<eagle version="6.5.0">
+<eagle version="6.6.0">
 <drawing>
 <settings>
@@
 <attribute name="NAME" x="12.2834" y="27.5272" size="0.8128" layer="26" font="vector" rot="MR180"/>
 </element>
-<element name="U1" library="Voltage-Reg" package="SOT23" value="TS5204" x="0" y="31.115" smashed="yes" rot="MR180">
+<element name="U1" library="Voltage-Reg" package="SOT23" value="TS5204-3V3" x="0" y="31.115" smashed="yes" rot="MR180">
 <attribute name="NAME" x="-0.635" y="28.8291" size="0.8128" layer="26" font="vector" rot="MR180"/>
 <attribute name="VALUE" x="-2.2225" y="27.6859" size="0.8128" layer="28" font="vector" rot="MR180"/>
