File: pcb/MI0283QT_v12b.sch (EAGLE design)
At the start: 36 parts, among them IC1 ADS7846, IC2 74LVC244, Q1 N-CHN, U1 TS5204, X1 PASSER, X2 PASSER, X3 PASSER, X4 PASSER

Commit message: updated cad files to Eagle xml format
Parts:
- removed ID: (no value), jumper:SJ2W
- added BUSY-RS, IM0, IM1: (no value), jumper:SJ2W
Connections:
- removed net A-LCD_LED: CON1.5, IC2A.A3, R8.1
- new net A-LCD_RS: BUSY-RS.3, IC2A.A3
- new net LCD_RS: IC2A.Y3, LCD.!WR!/SCL
- new net N$2: BUSY-RS.2, CON1.12
- new net N$4: IM1.2, LCD.IM3
- net +3V3: now also IM0.3, IM1.3; no longer ID.3
- net ADS_BUSY: now also BUSY-RS.1; no longer CON1.12
- net GND: now also IM0.1, IM1.1; no longer CON2.1, CON2.2, CON2.3, CON2.4, CON2.8, ID.1, LCD.!WR!/SCL, LCD.IM3
- net IM0: now also IM0.2; no longer ID.2
- net LCD_LED: now also CON1.5, R8.1; no longer IC2A.Y3
Other:
- note added: "8bit 0 1 1 0"
- note added: "9bit 0 1 0 1"
- note added: "SPI IM3 IM2 IM1 IM0"
- moved on the sheet: CON2, R8

Commit message: updated license infos
Other:
- note added: "Released under the Creative Commons Attribution Share-Alike License"
- note added: "http://creativecommons.org/licenses/by-sa/4.0/"
- note removed: "Released under the Creative Commons Attribution Share-Alike 3.0 License"
- note removed: "http://creativecommons.org/licenses/by-sa/3.0/"
Changed lines of the file:
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@@
 <text x="45.085" y="149.225" size="1.778" layer="95">1</text>
 <text x="45.085" y="141.605" size="1.778" layer="95">0</text>
-<text x="161.29" y="31.75" size="1.27" layer="95">Released under the Creative Commons Attribution Share-Alike 3.0 License</text>
-<text x="161.29" y="29.21" size="1.27" layer="95">http://creativecommons.org/licenses/by-sa/3.0/</text>
+<text x="161.29" y="31.75" size="1.27" layer="95">Released under the Creative Commons Attribution Share-Alike License</text>
+<text x="161.29" y="29.21" size="1.27" layer="95">http://creativecommons.org/licenses/by-sa/4.0/</text>
 <text x="161.29" y="25.4" size="1.27" layer="95">Designed by Andreas Watterott (Watterott electronic)</text>
 <text x="44.45" y="166.37" size="3.81" layer="250">Display</text>

Commit message: updated schematic and layout files
Parts:
- U1: value TS5204 -> TS5204-3V3
Changed lines of the file:
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@@
 <?xml version="1.0" encoding="utf-8"?>
 <!DOCTYPE eagle SYSTEM "eagle.dtd">
-<eagle version="6.5.0">
+<eagle version="6.6.0">
 <drawing>
 <settings>
@@
 <part name="R3" library="rcl" deviceset="R-EU_" device="R0603" value="47"/>
 <part name="R4" library="rcl" deviceset="R-EU_" device="R0603" value="47"/>
-<part name="U1" library="Voltage-Reg" deviceset="TS5204" device=""/>
+<part name="U1" library="Voltage-Reg" deviceset="TS5204" device="" value="TS5204-3V3"/>
 <part name="+3V6" library="supply1" deviceset="+3V3" device=""/>
 <part name="GND9" library="supply1" deviceset="GND" device=""/>
