File: pcb/MI0283QT_v13.brd (EAGLE design)
At the start: 52 x 85 mm, 38 parts, among them IC1 ADS7846, IC2 74LVC244, T1 N-CHN, U1 TS5204, X1 PASSER, X2 PASSER, X3 PASSER, X4 PASSER

Commit message: updated license infos
Parts:
- R1, R2, R3, R4: value 22 -> 47
Routing:
- net GND: track 77.1 -> 2.50 mm
Changed lines of the file:
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@@
 </autorouter>
 <elements>
-<element name="R1" library="rcl" package="R0603" value="22" x="13.97" y="32.5438" smashed="yes" rot="MR90">
+<element name="R1" library="rcl" package="R0603" value="47" x="13.97" y="32.5438" smashed="yes" rot="MR90">
 <attribute name="NAME" x="13.1763" y="30.7976" size="0.8128" layer="26" font="vector" ratio="10" rot="MR180"/>
 </element>
-<element name="R2" library="rcl" package="R0603" value="22" x="12.065" y="32.5438" smashed="yes" rot="MR90">
+<element name="R2" library="rcl" package="R0603" value="47" x="12.065" y="32.5438" smashed="yes" rot="MR90">
 <attribute name="NAME" x="11.2713" y="30.7976" size="0.8128" layer="26" font="vector" ratio="10" rot="MR180"/>
 </element>
-<element name="R3" library="rcl" package="R0603" value="22" x="10.16" y="32.5438" smashed="yes" rot="MR90">
+<element name="R3" library="rcl" package="R0603" value="47" x="10.16" y="32.5438" smashed="yes" rot="MR90">
 <attribute name="NAME" x="9.3663" y="30.7976" size="0.8128" layer="26" font="vector" ratio="10" rot="MR180"/>
 </element>
-<element name="R4" library="rcl" package="R0603" value="22" x="8.255" y="32.5438" smashed="yes" rot="MR90">
+<element name="R4" library="rcl" package="R0603" value="47" x="8.255" y="32.5438" smashed="yes" rot="MR90">
 <attribute name="NAME" x="7.4613" y="30.7975" size="0.8128" layer="26" font="vector" ratio="10" rot="MR180"/>
 </element>
@@
 <contactref element="IM0" pad="1"/>
 <contactref element="IM1" pad="1"/>
-<wire x1="-14.295" y1="33.9122" x2="-14.295" y2="32.402" width="0.254" layer="16"/>
-<wire x1="-14.295" y1="32.402" x2="-14.478" y2="32.219" width="0.254" layer="16"/>
-<wire x1="-12.25" y1="28.6825" x2="-11.75" y2="28.6825" width="0.254" layer="16"/>
-<wire x1="-11.75" y1="28.6825" x2="-11.25" y2="28.6825" width="0.254" layer="16"/>
-<wire x1="-8.75" y1="28.6825" x2="-8.75" y2="27.572" width="0.254" layer="16"/>
-<wire x1="-8.75" y1="27.572" x2="-8.89" y2="27.432" width="0.254" layer="16"/>
-<wire x1="-8.89" y1="27.432" x2="-11.049" y2="27.432" width="0.254" layer="16"/>
-<wire x1="-11.049" y1="27.432" x2="-11.25" y2="27.633" width="0.254" layer="16"/>
-<wire x1="-11.25" y1="28.6825" x2="-11.25" y2="27.633" width="0.254" layer="16"/>
-<wire x1="-8.636" y1="26.035" x2="-8.89" y2="26.289" width="0.254" layer="16"/>
-<wire x1="-8.89" y1="26.289" x2="-8.89" y2="27.432" width="0.254" layer="16"/>
-<wire x1="0.75" y1="28.6825" x2="1.25" y2="28.6825" width="0.254" layer="16"/>
-<wire x1="1.75" y1="28.6825" x2="2.25" y2="28.6825" width="0.254" layer="16"/>
-<wire x1="3.25" y1="28.6825" x2="3.75" y2="28.6825" width="0.254" layer="16"/>
-<wire x1="4.75" y1="28.6825" x2="5.25" y2="28.6825" width="0.254" layer="16"/>
-<wire x1="5.75" y1="28.6825" x2="6.25" y2="28.6825" width="0.254" layer="16"/>
-<wire x1="6.25" y1="28.6825" x2="6.75" y2="28.6825" width="0.254" layer="16"/>
-<wire x1="6.75" y1="28.6825" x2="7.25" y2="28.6825" width="0.254" layer="16"/>
 <wire x1="7.239" y1="28.6715" x2="7.25" y2="28.6825" width="0.254" layer="16"/>
-<wire x1="0.75" y1="28.6825" x2="0.75" y2="27.293" width="0.254" layer="16"/>
-<wire x1="0.762" y1="26.035" x2="-4.826" y2="26.035" width="0.254" layer="16"/>
-<wire x1="-4.826" y1="26.035" x2="-7.366" y2="26.035" width="0.254" layer="16"/>
-<wire x1="-7.366" y1="26.035" x2="-8.636" y2="26.035" width="0.254" layer="16"/>
-<wire x1="9.25" y1="28.6825" x2="9.25" y2="29.485" width="0.254" layer="16"/>
-<wire x1="9.25" y1="29.485" x2="8.128" y2="30.607" width="0.254" layer="16"/>
-<wire x1="8.128" y1="30.607" x2="7.747" y2="30.607" width="0.254" layer="16"/>
-<wire x1="7.747" y1="30.607" x2="7.493" y2="30.861" width="0.254" layer="16"/>
-<wire x1="7.493" y1="30.861" x2="6.477" y2="30.861" width="0.254" layer="16"/>
-<wire x1="6.477" y1="30.861" x2="6.223" y2="30.607" width="0.254" layer="16"/>
-<wire x1="6.223" y1="30.607" x2="6.223" y2="28.7095" width="0.254" layer="16"/>
 <wire x1="6.223" y1="28.7095" x2="6.25" y2="28.6825" width="0.254" layer="16"/>
-<wire x1="19.5825" y1="33.3375" x2="19.5825" y2="31.4213" width="0.254" layer="16"/>
 <wire x1="19.5825" y1="31.4213" x2="19.6825" y2="31.3213" width="0.254" layer="16"/>
-<wire x1="0.0508" y1="38.1" x2="3.556" y2="38.1" width="0.4064" layer="16"/>
-<wire x1="3.556" y1="38.1" x2="4.191" y2="37.465" width="0.4064" layer="16"/>
-<wire x1="4.191" y1="37.465" x2="4.191" y2="36.234" width="0.4064" layer="16"/>
 <wire x1="4.191" y1="36.234" x2="4.23" y2="36.195" width="0.4064" layer="16"/>
-<wire x1="-18.7253" y1="37.973" x2="-18.7253" y2="35.0837" width="0.254" layer="16"/>
 <wire x1="-18.7253" y1="35.0837" x2="-18.757" y2="35.052" width="0.254" layer="16"/>
-<wire x1="-14.478" y1="32.219" x2="-14.058" y2="32.219" width="0.254" layer="16"/>
-<wire x1="-14.058" y1="32.219" x2="-12.319" y2="30.48" width="0.254" layer="16"/>
-<wire x1="-12.319" y1="30.48" x2="-12.319" y2="28.7515" width="0.254" layer="16"/>
 <wire x1="-12.319" y1="28.7515" x2="-12.25" y2="28.6825" width="0.254" layer="16"/>
 <via x="21.717" y="36.449" extent="1-16" drill="0.3" shape="octagon"/>
 <via x="21.717" y="31.242" extent="1-16" drill="0.3" shape="octagon"/>
 <wire x1="19.7618" y1="31.242" x2="19.6825" y2="31.3213" width="0.254" layer="16"/>
-<wire x1="1.25" y1="28.6825" x2="1.75" y2="28.6825" width="0.254" layer="16"/>
-<wire x1="2.25" y1="28.6825" x2="2.75" y2="28.6825" width="0.254" layer="16"/>
-<wire x1="2.75" y1="28.6825" x2="3.25" y2="28.6825" width="0.254" layer="16"/>
-<wire x1="3.75" y1="28.6825" x2="4.25" y2="28.6825" width="0.254" layer="16"/>
-<wire x1="4.25" y1="28.6825" x2="4.75" y2="28.6825" width="0.254" layer="16"/>
-<wire x1="5.25" y1="28.6825" x2="4.25" y2="28.6825" width="0.254" layer="16"/>
-<wire x1="5.75" y1="28.6825" x2="5.25" y2="28.6825" width="0.254" layer="16"/>
 <wire x1="6.75" y1="28.6825" x2="6.75" y2="28.594" width="0.254" layer="16"/>
 <wire x1="6.75" y1="28.594" x2="6.731" y2="28.575" width="0.254" layer="16"/>
-<wire x1="6.731" y1="28.575" x2="6.3575" y2="28.575" width="0.254" layer="16"/>
-<wire x1="6.3575" y1="28.575" x2="6.25" y2="28.6825" width="0.254" layer="16"/>
-<wire x1="-13.843" y1="35.306" x2="-14.224" y2="34.925" width="0.254" layer="16"/>
-<wire x1="-14.224" y1="34.925" x2="-14.224" y2="33.9832" width="0.254" layer="16"/>
-<wire x1="-14.224" y1="33.9832" x2="-14.295" y2="33.9122" width="0.254" layer="16"/>
-<wire x1="-18.7253" y1="35.0837" x2="-18.7253" y2="34.6003" width="0.254" layer="16"/>
-<wire x1="-18.7253" y1="34.6003" x2="-17.145" y2="33.02" width="0.254" layer="16"/>
 <via x="-17.145" y="33.02" extent="1-16" drill="0.3" shape="octagon"/>
-<wire x1="-17.145" y1="33.02" x2="-16.129" y2="33.02" width="0.254" layer="1"/>
-<wire x1="-16.129" y1="33.02" x2="-13.843" y2="35.306" width="0.254" layer="1"/>
 <via x="-13.843" y="35.306" extent="1-16" drill="0.3" shape="octagon"/>
 <wire x1="19.939" y1="23.241" x2="20.066" y2="23.241" width="0.254" layer="16"/>
@@
 <contactref element="LCD" pad="25"/>
 <contactref element="LCD" pad="35"/>
-<wire x1="-13.843" y1="35.306" x2="-11.938" y2="35.306" width="0.254" layer="1"/>
-<wire x1="-11.938" y1="35.306" x2="-9.144" y2="32.512" width="0.254" layer="1"/>
 <via x="-9.144" y="32.512" extent="1-16" drill="0.3" shape="octagon"/>
-<wire x1="-9.144" y1="32.512" x2="-8.0082" y2="32.512" width="0.254" layer="16"/>
-<wire x1="-8.0082" y1="32.512" x2="-7.9375" y2="32.4413" width="0.254" layer="16"/>
-<wire x1="-2.25" y1="28.6825" x2="-2.75" y2="28.6825" width="0.254" layer="16"/>
-<wire x1="0.25" y1="28.6825" x2="0.75" y2="28.6825" width="0.254" layer="16"/>
-<wire x1="0.25" y1="28.6825" x2="-0.25" y2="28.6825" width="0.254" layer="16"/>
-<wire x1="-0.25" y1="28.6825" x2="-0.75" y2="28.6825" width="0.254" layer="16"/>
-<wire x1="-0.75" y1="28.6825" x2="-1.25" y2="28.6825" width="0.254" layer="16"/>
-<wire x1="-1.25" y1="28.6825" x2="-1.75" y2="28.6825" width="0.254" layer="16"/>
-<wire x1="-1.75" y1="28.6825" x2="-2.25" y2="28.6825" width="0.254" layer="16"/>
-<wire x1="-2.75" y1="28.6825" x2="-3.25" y2="28.6825" width="0.254" layer="16"/>
-<wire x1="-6.75" y1="28.6825" x2="-6.75" y2="27.54" width="0.254" layer="16"/>
-<wire x1="-6.75" y1="27.54" x2="-7.366" y2="26.924" width="0.254" layer="16"/>
-<wire x1="-7.366" y1="26.924" x2="-7.366" y2="26.035" width="0.254" layer="16"/>
-<wire x1="-4.75" y1="28.6825" x2="-4.75" y2="26.111" width="0.254" layer="16"/>
-<wire x1="-4.75" y1="26.111" x2="-4.826" y2="26.035" width="0.254" layer="16"/>
 <wire x1="20.066" y1="23.241" x2="18.542" y2="23.241" width="0.15" layer="16"/>
 </signal>

Commit message: updated schematic and layout files
Parts:
- U1: value TS5204 -> TS5204-3V3
Changed lines of the file:
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@@
 <?xml version="1.0" encoding="utf-8"?>
 <!DOCTYPE eagle SYSTEM "eagle.dtd">
-<eagle version="6.5.0">
+<eagle version="6.6.0">
 <drawing>
 <settings>
@@
 <attribute name="NAME" x="7.4613" y="30.7975" size="0.8128" layer="26" font="vector" ratio="10" rot="MR180"/>
 </element>
-<element name="U1" library="Voltage-Reg" package="SOT23" value="TS5204" x="15.875" y="8.255" smashed="yes" rot="MR0">
+<element name="U1" library="Voltage-Reg" package="SOT23" value="TS5204-3V3" x="15.875" y="8.255" smashed="yes" rot="MR0">
 <attribute name="NAME" x="16.51" y="10.3188" size="0.8128" layer="26" font="vector" ratio="10" rot="MR0"/>
 </element>

Commit message: updated layout and schematics
Other:
- board text added: "Silkscreen: 22 bPlace + 26 bNames"
Changed lines of the file:
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@@
 <setting verticaltext="up"/>
 </settings>
-<grid distance="0.127" unitdist="mm" unit="mm" style="lines" multiple="1" display="yes" altdistance="0.00625" altunitdist="inch" altunit="inch"/>
+<grid distance="0.05" unitdist="inch" unit="inch" style="lines" multiple="1" display="yes" altdistance="0.0125" altunitdist="inch" altunit="inch"/>
 <layers>
 <layer number="1" name="Top" color="4" fill="1" visible="yes" active="yes"/>
@@
 <text x="4.8895" y="8.5725" size="0.8128" layer="22" font="vector" rot="MR0">Display</text>
 <text x="-4.953" y="8.5725" size="0.8128" layer="22" font="vector" rot="MR0">Touch</text>
+<text x="-25.4" y="-1.27" size="1.27" layer="49" font="vector" ratio="10" align="top-left">Silkscreen: 22 bPlace + 26 bNames</text>
 </plain>
 <attributes>

Commit message: cleaned up schematics and layout
Parts:
- removed R16: 100k, rcl:R0603
Connections:
- net GND: no longer R16.2
Changed lines of the file:
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@@
 <layer number="48" name="Document" color="7" fill="1" visible="yes" active="yes"/>
 <layer number="49" name="Reference" color="7" fill="1" visible="yes" active="yes"/>
-<layer number="50" name="dxf" color="7" fill="1" visible="yes" active="yes"/>
 <layer number="51" name="tDocu" color="7" fill="1" visible="yes" active="yes"/>
 <layer number="52" name="bDocu" color="7" fill="1" visible="yes" active="yes"/>
 <layer number="53" name="tCopper" color="7" fill="11" visible="no" active="no"/>
 <layer number="54" name="bCopper" color="7" fill="1" visible="no" active="no"/>
-<layer number="56" name="wert" color="7" fill="1" visible="yes" active="yes"/>
 <layer number="91" name="Nets" color="2" fill="1" visible="no" active="no"/>
 <layer number="92" name="Busses" color="1" fill="1" visible="no" active="no"/>
@@
 <layer number="98" name="Guide" color="6" fill="1" visible="no" active="no"/>
 <layer number="100" name="Muster" color="7" fill="1" visible="no" active="no"/>
-<layer number="101" name="Bemassung" color="7" fill="1" visible="yes" active="yes"/>
-<layer number="102" name="fp2" color="7" fill="1" visible="yes" active="yes"/>
-<layer number="103" name="fp3" color="7" fill="1" visible="yes" active="yes"/>
-<layer number="104" name="fp4" color="7" fill="1" visible="yes" active="yes"/>
-<layer number="105" name="fp5" color="7" fill="1" visible="yes" active="yes"/>
-<layer number="106" name="fp6" color="7" fill="1" visible="yes" active="yes"/>
-<layer number="107" name="fp7" color="7" fill="1" visible="yes" active="yes"/>
-<layer number="108" name="fp8" color="7" fill="1" visible="yes" active="yes"/>
-<layer number="109" name="fp9" color="7" fill="1" visible="yes" active="yes"/>
-<layer number="110" name="fp0" color="7" fill="1" visible="yes" active="yes"/>
-<layer number="116" name="Patch_BOT" color="9" fill="4" visible="yes" active="yes"/>
-<layer number="120" name="Descript" color="7" fill="1" visible="yes" active="yes"/>
-<layer number="121" name="tTestdril" color="7" fill="1" visible="yes" active="yes"/>
-<layer number="122" name="bTestdril" color="7" fill="1" visible="yes" active="yes"/>
-<layer number="123" name="tTestmark" color="7" fill="1" visible="yes" active="yes"/>
-<layer number="124" name="bTestmark" color="7" fill="1" visible="yes" active="yes"/>
-<layer number="144" name="DrillLegend" color="7" fill="1" visible="yes" active="yes"/>
-<layer number="151" name="HeatSink" color="7" fill="1" visible="yes" active="yes"/>
-<layer number="200" name="200bmp" color="1" fill="10" visible="yes" active="yes"/>
-<layer number="201" name="201bmp" color="2" fill="10" visible="yes" active="yes"/>
-<layer number="202" name="202bmp" color="3" fill="10" visible="yes" active="yes"/>
-<layer number="203" name="203bmp" color="4" fill="10" visible="yes" active="yes"/>
-<layer number="204" name="204bmp" color="5" fill="10" visible="yes" active="yes"/>
-<layer number="205" name="205bmp" color="6" fill="10" visible="yes" active="yes"/>
-<layer number="206" name="206bmp" color="7" fill="10" visible="yes" active="yes"/>
-<layer number="207" name="207bmp" color="15" fill="10" visible="yes" active="yes"/>
-<layer number="208" name="208bmp" color="9" fill="10" visible="yes" active="yes"/>
-<layer number="209" name="209bmp" color="7" fill="1" visible="yes" active="yes"/>
-<layer number="210" name="210bmp" color="7" fill="1" visible="yes" active="yes"/>
-<layer number="211" name="211bmp" color="7" fill="1" visible="yes" active="yes"/>
-<layer number="212" name="212bmp" color="7" fill="1" visible="yes" active="yes"/>
-<layer number="213" name="213bmp" color="7" fill="1" visible="yes" active="yes"/>
-<layer number="214" name="214bmp" color="7" fill="1" visible="yes" active="yes"/>
-<layer number="215" name="215bmp" color="7" fill="1" visible="yes" active="yes"/>
-<layer number="216" name="216bmp" color="7" fill="1" visible="yes" active="yes"/>
-<layer number="250" name="Descript" color="3" fill="1" visible="yes" active="yes"/>
 <layer number="251" name="SMDround" color="12" fill="11" visible="no" active="no"/>
-<layer number="254" name="OrgLBR" color="13" fill="1" visible="yes" active="yes"/>
 </layers>
 <board>
@@
 <attribute name="NAME" x="-10.922" y="42.672" size="0.8128" layer="26" rot="MR0"/>
 </element>
-<element name="R16" library="rcl" package="R0603" value="100k" x="-3.81" y="43.815" smashed="yes" rot="MR0">
-<attribute name="NAME" x="-5.334" y="43.434" size="0.8128" layer="26" rot="MR0"/>
-</element>
 <element name="VREF-3V3" library="jumper" package="SJ" value="" x="-13.335" y="3.175" smashed="yes" rot="MR180">
 <attribute name="NAME" x="-17.399" y="5.461" size="0.9" layer="26" font="vector" ratio="10" rot="MR180"/>
@@
 <contactref element="IC2" pad="10"/>
 <contactref element="C7" pad="2"/>
-<contactref element="R16" pad="2"/>
 <contactref element="R14" pad="2"/>
 <contactref element="IC2" pad="1"/>
