File: pcb/MI0283QT_v13.sch (EAGLE design)
At the start: 38 parts, among them IC1 ADS7846, IC2 74LVC244, T1 N-CHN, U1 TS5204, X1 PASSER, X2 PASSER, X3 PASSER, X4 PASSER

Commit message: updated license infos
Parts:
- R1, R2, R3, R4: value 22 -> 47
Other:
- note added: "Released under the Creative Commons Attribution Share-Alike License"
- note added: "http://creativecommons.org/licenses/by-sa/4.0/"
- note removed: "Released under the Creative Commons Attribution Share-Alike 3.0 License"
- note removed: "http://creativecommons.org/licenses/by-sa/3.0/"
Changed lines of the file:
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@@
 <parts>
 <part name="GND3" library="supply1" deviceset="GND" device=""/>
-<part name="R1" library="rcl" deviceset="R-EU_" device="R0603" value="22"/>
-<part name="R2" library="rcl" deviceset="R-EU_" device="R0603" value="22"/>
-<part name="R3" library="rcl" deviceset="R-EU_" device="R0603" value="22"/>
-<part name="R4" library="rcl" deviceset="R-EU_" device="R0603" value="22"/>
+<part name="R1" library="rcl" deviceset="R-EU_" device="R0603" value="47"/>
+<part name="R2" library="rcl" deviceset="R-EU_" device="R0603" value="47"/>
+<part name="R3" library="rcl" deviceset="R-EU_" device="R0603" value="47"/>
+<part name="R4" library="rcl" deviceset="R-EU_" device="R0603" value="47"/>
 <part name="U1" library="Voltage-Reg" deviceset="TS5204" device=""/>
 <part name="GND9" library="supply1" deviceset="GND" device=""/>
@@
 <text x="45.085" y="146.685" size="1.778" layer="95">1</text>
 <text x="45.085" y="139.065" size="1.778" layer="95">0</text>
-<text x="161.29" y="31.75" size="1.27" layer="95">Released under the Creative Commons Attribution Share-Alike 3.0 License</text>
-<text x="161.29" y="29.21" size="1.27" layer="95">http://creativecommons.org/licenses/by-sa/3.0/</text>
+<text x="161.29" y="31.75" size="1.27" layer="95">Released under the Creative Commons Attribution Share-Alike License</text>
+<text x="161.29" y="29.21" size="1.27" layer="95">http://creativecommons.org/licenses/by-sa/4.0/</text>
 <text x="161.29" y="25.4" size="1.27" layer="95">Designed by Andreas Watterott (Watterott electronic)</text>
 <text x="26.67" y="166.37" size="3.81" layer="250">Display with Touch-Panel</text>

Commit message: updated schematics
Other:
- note added: "8bit x 1 1 0"
- note added: "9bit x 1 0 1"
- note added: "Jumper IM1 is IM3"
- note removed: "8bit 0 1 1 0"
- note removed: "9bit 0 1 0 1"
Changed lines of the file:
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@@
 <setting verticaltext="up"/>
 </settings>
-<grid distance="0.1" unitdist="inch" unit="inch" style="lines" multiple="1" display="no" altdistance="0.01" altunitdist="inch" altunit="inch"/>
+<grid distance="0.05" unitdist="inch" unit="inch" style="lines" multiple="1" display="yes" altdistance="0.01" altunitdist="inch" altunit="inch"/>
 <layers>
 <layer number="1" name="Top" color="4" fill="1" visible="no" active="no"/>
@@
 <wire x1="27.94" y1="142.24" x2="27.94" y2="140.335" width="0.8128" layer="94"/>
 <wire x1="232.41" y1="50.292" x2="232.41" y2="48.26" width="0.4064" layer="94"/>
-<text x="46.99" y="158.75" size="1.27" layer="250" font="vector">9bit  0   1   0   1</text>
-<text x="46.99" y="156.21" size="1.27" layer="250" font="vector">8bit  0   1   1   0</text>
+<text x="46.99" y="158.75" size="1.27" layer="250" font="vector">9bit  x   1   0   1</text>
+<text x="46.99" y="156.21" size="1.27" layer="250" font="vector">8bit  x   1   1   0</text>
 <text x="46.99" y="161.29" size="1.27" layer="250" font="vector">SPI  IM3 IM2 IM1 IM0</text>
+<text x="19.05" y="156.21" size="1.6764" layer="250" font="vector">Jumper IM1 is IM3</text>
+<wire x1="31.75" y1="156.21" x2="29.21" y2="144.78" width="0.1524" layer="250"/>
 </plain>
 <instances>

Commit message: updated schematic and layout files
Parts:
- U1: value TS5204 -> TS5204-3V3
Changed lines of the file:
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@@
 <?xml version="1.0" encoding="utf-8"?>
 <!DOCTYPE eagle SYSTEM "eagle.dtd">
-<eagle version="6.5.0">
+<eagle version="6.6.0">
 <drawing>
 <settings>
@@
 <setting verticaltext="up"/>
 </settings>
-<grid distance="0.05" unitdist="inch" unit="inch" style="lines" multiple="1" display="yes" altdistance="0.01" altunitdist="inch" altunit="inch"/>
+<grid distance="0.1" unitdist="inch" unit="inch" style="lines" multiple="1" display="no" altdistance="0.01" altunitdist="inch" altunit="inch"/>
 <layers>
 <layer number="1" name="Top" color="4" fill="1" visible="no" active="no"/>
@@
 <part name="R3" library="rcl" deviceset="R-EU_" device="R0603" value="47"/>
 <part name="R4" library="rcl" deviceset="R-EU_" device="R0603" value="47"/>
-<part name="U1" library="Voltage-Reg" deviceset="TS5204" device=""/>
+<part name="U1" library="Voltage-Reg" deviceset="TS5204" device="" value="TS5204-3V3"/>
 <part name="GND9" library="supply1" deviceset="GND" device=""/>
 <part name="VCC-3V3" library="jumper" deviceset="SJ" device=""/>

Commit message: cleaned up schematics and layout
Parts:
- removed R16: 100k, rcl:R-EU_R0603
Connections:
- net GND: no longer R16.2
Changed lines of the file:
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@@
 <layer number="98" name="Guide" color="6" fill="1" visible="yes" active="yes"/>
 <layer number="100" name="Muster" color="7" fill="1" visible="no" active="no"/>
-<layer number="101" name="Bemassung" color="7" fill="1" visible="yes" active="yes"/>
-<layer number="102" name="fp2" color="7" fill="1" visible="yes" active="yes"/>
-<layer number="103" name="fp3" color="7" fill="1" visible="yes" active="yes"/>
-<layer number="104" name="fp4" color="7" fill="1" visible="yes" active="yes"/>
-<layer number="105" name="fp5" color="7" fill="1" visible="yes" active="yes"/>
-<layer number="106" name="fp6" color="7" fill="1" visible="yes" active="yes"/>
-<layer number="107" name="fp7" color="7" fill="1" visible="yes" active="yes"/>
-<layer number="108" name="fp8" color="7" fill="1" visible="yes" active="yes"/>
-<layer number="109" name="fp9" color="7" fill="1" visible="yes" active="yes"/>
-<layer number="110" name="fp0" color="7" fill="1" visible="yes" active="yes"/>
-<layer number="116" name="Patch_BOT" color="9" fill="4" visible="yes" active="yes"/>
-<layer number="120" name="Descript" color="7" fill="1" visible="yes" active="yes"/>
-<layer number="121" name="tTestdril" color="7" fill="1" visible="yes" active="yes"/>
-<layer number="122" name="bTestdril" color="7" fill="1" visible="yes" active="yes"/>
-<layer number="123" name="tTestmark" color="7" fill="1" visible="yes" active="yes"/>
-<layer number="124" name="bTestmark" color="7" fill="1" visible="yes" active="yes"/>
-<layer number="144" name="DrillLegend" color="7" fill="1" visible="yes" active="yes"/>
-<layer number="151" name="HeatSink" color="7" fill="1" visible="yes" active="yes"/>
-<layer number="200" name="200bmp" color="1" fill="10" visible="yes" active="yes"/>
-<layer number="201" name="201bmp" color="2" fill="10" visible="yes" active="yes"/>
-<layer number="202" name="202bmp" color="3" fill="10" visible="yes" active="yes"/>
-<layer number="203" name="203bmp" color="4" fill="10" visible="yes" active="yes"/>
-<layer number="204" name="204bmp" color="5" fill="10" visible="yes" active="yes"/>
-<layer number="205" name="205bmp" color="6" fill="10" visible="yes" active="yes"/>
-<layer number="206" name="206bmp" color="7" fill="10" visible="yes" active="yes"/>
-<layer number="207" name="207bmp" color="15" fill="10" visible="yes" active="yes"/>
-<layer number="208" name="208bmp" color="9" fill="10" visible="yes" active="yes"/>
-<layer number="209" name="209bmp" color="7" fill="1" visible="yes" active="yes"/>
-<layer number="210" name="210bmp" color="7" fill="1" visible="yes" active="yes"/>
-<layer number="211" name="211bmp" color="7" fill="1" visible="yes" active="yes"/>
-<layer number="212" name="212bmp" color="7" fill="1" visible="yes" active="yes"/>
-<layer number="213" name="213bmp" color="7" fill="1" visible="yes" active="yes"/>
-<layer number="214" name="214bmp" color="7" fill="1" visible="yes" active="yes"/>
-<layer number="215" name="215bmp" color="7" fill="1" visible="yes" active="yes"/>
-<layer number="216" name="216bmp" color="7" fill="1" visible="yes" active="yes"/>
 <layer number="250" name="Descript" color="3" fill="1" visible="yes" active="yes"/>
 <layer number="251" name="SMDround" color="12" fill="11" visible="no" active="no"/>
-<layer number="254" name="OrgLBR" color="13" fill="1" visible="yes" active="yes"/>
 </layers>
 <schematic xreflabel="%F%N/%S.%C%R" xrefpart="/%S.%C%R">
@@
 <part name="R14" library="rcl" deviceset="R-EU_" device="R0603" value="100k"/>
 <part name="R15" library="rcl" deviceset="R-EU_" device="R0603" value="100k"/>
-<part name="R16" library="rcl" deviceset="R-EU_" device="R0603" value="100k"/>
 <part name="+3V1" library="supply1" deviceset="+3V3" device=""/>
 <part name="+3V5" library="supply1" deviceset="+3V3" device=""/>
 <part name="+3V12" library="supply1" deviceset="+3V3" device=""/>
 <part name="+3V13" library="supply1" deviceset="+3V3" device=""/>
-<part name="GND14" library="supply1" deviceset="GND" device=""/>
 <part name="GND15" library="supply1" deviceset="GND" device=""/>
 <part name="VREF-3V3" library="jumper" deviceset="SJ" device=""/>
@@
 <attribute name="VALUE" x="193.04" y="105.029" size="1.778" layer="96" rot="MR90"/>
 </instance>
-<instance part="R16" gate="G$1" x="199.39" y="130.81" smashed="yes" rot="MR270">
-<attribute name="NAME" x="198.0184" y="132.588" size="1.778" layer="95" rot="MR270"/>
-<attribute name="VALUE" x="200.66" y="128.905" size="1.778" layer="96" rot="MR90"/>
-</instance>
 <instance part="+3V1" gate="G$1" x="191.77" y="158.75" smashed="yes" rot="MR0">
 <attribute name="VALUE" x="189.23" y="161.29" size="1.778" layer="96" rot="MR180"/>
@@
 <instance part="+3V13" gate="G$1" x="199.39" y="115.57" smashed="yes" rot="MR0">
 <attribute name="VALUE" x="196.85" y="118.11" size="1.778" layer="96" rot="MR180"/>
-</instance>
-<instance part="GND14" gate="1" x="199.39" y="123.19" smashed="yes" rot="MR0">
-<attribute name="VALUE" x="201.93" y="120.65" size="1.778" layer="96" rot="MR0"/>
 </instance>
 <instance part="GND15" gate="1" x="199.39" y="80.01" smashed="yes" rot="MR0">
@@
 </segment>
 <segment>
-<pinref part="R16" gate="G$1" pin="2"/>
-<pinref part="GND14" gate="1" pin="GND"/>
-</segment>
-<segment>

Commit message: cleaned up schematics and layout
Changed lines of the file:
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@@
 <setting verticaltext="up"/>
 </settings>
-<grid distance="0.1" unitdist="inch" unit="inch" style="lines" multiple="1" display="no" altdistance="0.01" altunitdist="inch" altunit="inch"/>
+<grid distance="0.05" unitdist="inch" unit="inch" style="lines" multiple="1" display="yes" altdistance="0.025" altunitdist="inch" altunit="inch"/>
 <layers>
 <layer number="1" name="Top" color="4" fill="1" visible="no" active="no"/>
@@
 <part name="R5" library="rcl" deviceset="R-EU_" device="R0603" value="47"/>
 <part name="P+1" library="supply1" deviceset="VCC" device=""/>
-<part name="FRAME1" library="frames" deviceset="A4L-LOC" device=""/>
 <part name="C6" library="rcl" deviceset="C-EU" device="C0603" value="100nF"/>
 <part name="GND17" library="supply1" deviceset="GND" device=""/>
@@
 <part name="IM1" library="jumper" deviceset="SJ2W" device=""/>
 <part name="BUSY-RS" library="jumper" deviceset="SJ2W" device=""/>
+<part name="FRAME1" library="we-symbol" deviceset="FRAME-A4L" device=""/>
 </parts>
 <sheets>
@@
 <text x="45.085" y="146.685" size="1.778" layer="95">1</text>
 <text x="45.085" y="139.065" size="1.778" layer="95">0</text>
-<text x="161.29" y="31.75" size="1.27" layer="95">Released under the Creative Commons Attribution Share-Alike License</text>
-<text x="161.29" y="29.21" size="1.27" layer="95">http://creativecommons.org/licenses/by-sa/4.0/</text>
-<text x="161.29" y="25.4" size="1.27" layer="95">Designed by Andreas Watterott (Watterott electronic)</text>
+<text x="162.56" y="21.59" size="1.27" layer="95">Released under the Creative Commons Attribution Share-Alike License</text>
+<text x="162.56" y="19.05" size="1.27" layer="95">http://creativecommons.org/licenses/by-sa/4.0/</text>
+<text x="162.56" y="15.24" size="1.27" layer="95">Designed by Andreas Watterott (Watterott electronic)</text>
 <text x="26.67" y="166.37" size="3.81" layer="250">Display with Touch-Panel</text>
 <wire x1="105.41" y1="65.024" x2="105.41" y2="67.183" width="0.8128" layer="94"/>
@@
 <attribute name="VALUE" x="102.87" y="111.76" size="1.778" layer="96" rot="R90"/>
 </instance>
-<instance part="FRAME1" gate="G$1" x="0" y="0" smashed="yes">
-<attribute name="DRAWING_NAME" x="217.17" y="15.24" size="2.54" layer="94" font="vector"/>
-<attribute name="LAST_DATE_TIME" x="217.17" y="10.16" size="2.286" layer="94" font="vector"/>
-<attribute name="SHEET" x="230.505" y="5.08" size="2.54" layer="94" font="vector"/>
-</instance>
 <instance part="C6" gate="G$1" x="95.25" y="110.49" smashed="yes">
 <attribute name="NAME" x="96.012" y="110.871" size="1.778" layer="95"/>
@@
 <attribute name="VALUE" x="92.71" y="100.33" size="1.778" layer="96"/>
 </instance>
-<instance part="X1" gate="G$1" x="166.37" y="19.05"/>
-<instance part="X2" gate="G$1" x="173.99" y="19.05"/>
-<instance part="X3" gate="G$1" x="181.61" y="19.05"/>
-<instance part="X4" gate="G$1" x="189.23" y="19.05"/>
-<instance part="U$1" gate="G$1" x="201.93" y="19.05"/>
-<instance part="LOGO1" gate="G$1" x="201.93" y="11.43"/>
+<instance part="X1" gate="G$1" x="165.1" y="7.62" smashed="yes"/>
+<instance part="X2" gate="G$1" x="170.18" y="7.62" smashed="yes"/>
+<instance part="X3" gate="G$1" x="175.26" y="7.62" smashed="yes"/>
+<instance part="X4" gate="G$1" x="180.34" y="7.62" smashed="yes"/>
+<instance part="U$1" gate="G$1" x="208.28" y="7.62"/>
+<instance part="LOGO1" gate="G$1" x="198.12" y="7.62"/>
 <instance part="LCD" gate="G$1" x="57.15" y="104.14"/>
 <instance part="P+6" gate="VCC" x="107.95" y="29.21" smashed="yes">
@@
 <attribute name="VALUE" x="234.95" y="46.355" size="1.778" layer="96"/>
 </instance>
+<instance part="FRAME1" gate="G$1" x="0" y="0"/>
 </instances>
 <busses>
