File: hardware/MI0283QT_v15.brd (EAGLE design)
At the start: 52 x 85 mm, 38 parts, among them IC1 ADS7846PW, IC2 74244PW, IC3 VREG-TS9011-3V3, J1 MA08-2, J2 MA08-1, T1 N-Chn, X1 PASSER-07, X2 PASSER-07, X3 PASSER-07, X4 PASSER-07

Commit message: update schematics
Parts:
- renumbered BUSY-RS to RS-BUSY
Connections:
- net N$6 renamed BUSY_RS
Changed lines of the file:
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@@
 <attribute name="VALUE" x="12.54125" y="38.735" size="0.8128" layer="28" font="vector" ratio="10" rot="MR180" align="center"/>
 </element>
-<element name="BUSY-RS" library="we-rcl" package="JUMPER3-0603" value="JUMPER3-0603" x="-1.27" y="47.9425" smashed="yes" rot="MR270">
+<element name="RS-BUSY" library="we-rcl" package="JUMPER3-0603" value="JUMPER3-0603" x="-1.27" y="47.9425" smashed="yes" rot="MR270">
 <attribute name="NAME" x="-1.27" y="49.8475" size="1.016" layer="22" font="vector" ratio="12" rot="MR0" align="center"/>
 </element>
@@
 <signal name="ADS_BUSY">
 <contactref element="IC2" pad="5"/>
-<contactref element="BUSY-RS" pad="1"/>
+<contactref element="RS-BUSY" pad="1"/>
 <wire x1="-1.595" y1="44.91" x2="-1.595" y2="46.045" width="0.254" layer="16"/>
 <wire x1="-1.595" y1="46.045" x2="-2.67" y2="47.12" width="0.254" layer="16"/>
@@
 <signal name="A-LCD_RS">
 <contactref element="IC2" pad="6"/>
-<contactref element="BUSY-RS" pad="3"/>
+<contactref element="RS-BUSY" pad="3"/>
 <wire x1="0.13" y1="47.9425" x2="0.13" y2="47.12" width="0.254" layer="16"/>
 <wire x1="0.13" y1="47.12" x2="-0.945" y2="46.045" width="0.254" layer="16"/>
 <wire x1="-0.945" y1="44.91" x2="-0.945" y2="46.045" width="0.254" layer="16"/>
 </signal>
-<signal name="N$6">
-<contactref element="BUSY-RS" pad="2"/>
+<signal name="BUSY_RS">
+<contactref element="RS-BUSY" pad="2"/>
 <contactref element="J1" pad="12"/>
 <wire x1="-3.81" y1="3.175" x2="-5.08" y2="4.445" width="0.254" layer="16"/>
